File: 2164VCA/2164_VCA_PANEL/2164_VCA_PANEL.kicad_pcb (KiCad board)
At the start: 2 copper layers, 70.8 x 128.5 mm, 18 parts

Commit message: update vca panel
Parts:
- moved REF** 1.69 mm to (83.2, 120.0)
- moved REF** 1.17 mm to (116.7, 120.0)
